Commit message: nothingburger

File: dual_arm_workcell_moveit_config/config/dual_arm_workcell.ros2_control.xacro (robot description, xacro)
@@ -1,5 +1,5 @@
 <?xml version="1.0"?>
 <robot xmlns:xacro="http://www.ros.org/wiki/xacro">
-    <xacro:macro name="left_ur16e_ros2_control" params="name initial_positions_file">
+    <xacro:macro name="dual_arm_workcell_ros2_control" params="name initial_positions_file">
         <xacro:property name="initial_positions" value="${load_yaml(initial_positions_file)['initial_positions']}"/>
         <ros2_control name="${name}" type="system">
