Commit message: Everything left camera, right camera and dual robot system calibration is finished, only tool calibration is tbd

File: dual_arm_workcell_description/urdf/dual_arm_workcell.urdf.xacro (robot description, xacro)
@@ -152,5 +152,5 @@
      trajectory_port="$(arg left_trajectory_port)"
      >
-     <origin xyz="0 1.0 0" rpy="0 0 0" />          <!-- position robot in the world -->
+     <origin xyz="-0.236 0.555 -0.007" rpy="0.035 0.036 1.558" />          <!-- position robot in the world -->
    </xacro:ur_robot>
    <!-- right arm -->
@@ -192,5 +192,5 @@
      trajectory_port="$(arg right_trajectory_port)"
      >
-     <origin xyz="0 -1.0 0" rpy="0 0 0" />          <!-- position robot in the world -->
+     <origin xyz="0.635 0.594 0.010" rpy="-0.009 0.015 1.580" />          <!-- position robot in the world -->
    </xacro:ur_robot>
    <xacro:if value="$(arg sim_gazebo)">

Commit message: recalibrated the entire system, its pretty well done this time

File: dual_arm_workcell_description/urdf/dual_arm_workcell.urdf.xacro (robot description, xacro)
@@ -155,5 +155,5 @@
      trajectory_port="$(arg left_trajectory_port)"
      >
-     <origin xyz="-0.236 0.555 -0.007" rpy="0.035 0.036 1.558" />          <!-- position robot in the world -->
+     <origin xyz="-0.331 0.529 0.006" rpy="0.0 0.0 1.570796" />          <!-- position robot in the world -->
    </xacro:ur_robot>
    <!-- right arm -->
@@ -198,5 +198,5 @@
      trajectory_port="$(arg right_trajectory_port)"
      >
-     <origin xyz="0.635 0.594 0.010" rpy="-0.009 0.015 1.580" />          <!-- position robot in the world -->
+     <origin xyz="0.587 0.542 0.001" rpy="-0.00 0.0 1.570796" />          <!-- position robot in the world -->
    </xacro:ur_robot>
    <xacro:if value="$(arg sim_gazebo)">
